File: regua-pcb-fritzenlab.kicad_pcb (KiCad board)
At the start: 2 copper layers, 206 x 30 mm, 13 parts, among them J1 Conn_01x06_Pin, SW1 SW_Push_Dual, U1 ATtiny85-20S

Commit message: finished design, gerbers generated
Parts:
- removed the G*** at (246.6, 92.4)
- added G***: LOGO, logo:logo-35mm, F.Cu at (239.2, 89.4)
- moved BT1 2.19 mm to (98.8, 88.7)
Routing:
- net Net-(BT1-+): track 0.00 -> 62.0 mm
- net VCC: track 0.00 -> 56.4 mm, vias 0 -> 2
- net LED-unitario: track 0.00 -> 34.0 mm, vias 0 -> 2
- net Analog: track 0.00 -> 32.0 mm
- net LED-decimal: track 0.00 -> 29.3 mm, vias 0 -> 2
- net D10: track 0.00 -> 26.6 mm, vias 0 -> 2
- net GND: track 0.00 -> 16.7 mm, vias 0 -> 6
- net Net-(D1-K): track 0.00 -> 11.0 mm
- net REF: track 0.00 -> 6.30 mm
- added copper zone on B.Cu, net GND
Other:
- board text added: "0"
- board text added: "1"
- board text added: "10"
- board text added: "11"
- board text added: "12"
- board text added: "13"
- board text added: "14"
- board text added: "15"
- board text added: "16"
- board text added: "17"
- board text added: "18"
- board text added: "19"
- board text added: "2"
- board text added: "20"
- board text added: "3"
- board text added: "4"
- board text added: "5"
- board text added: "6"
- board text added: "7"
- board text added: "8"
- board text added: "9"
- board text added: "<- Attiny85 com bootloader Arduino, comece a hackear por aqui"
- board text added: "FritzenLab.net FritzenLab.com.br Loja.FritzenLab.com.br"
- board text added: "Led D1: dezena, Led D2: unidade. Ao pressionar o botão SW1, funciona assim: se D1 piscar duas vezes e D2 tres vezes, 23 graus. Se D1 nao piscar e D2 piscar oito vezes, 08 graus."
- board text added: "Pressione aqui (e segure)"
- board text added: "Regua termometro"
- board text added: "Termistor NTC ^^ 10k Ohm"

Commit message: backups
Parts:
- SW1: footprint Button_Switch_SMD:SW_SPST_PTS810 -> Button_Switch_SMD:SW_SPST_B3S-1000
- moved SW1 1.33 mm to (130.6, 82.2), turned to 0 degrees
Routing:
- net Net-(BT1-+): track 62.0 -> 66.7 mm
- net VCC: track 56.4 -> 58.2 mm
